File: mp3_fa2026.kicad_pcb (KiCad board)
At the start: 2 copper layers, 45.7 x 55 mm, 41 parts, among them J1 USB4105-GF-A, J2 LEFT, J3 RIGHT, J4 DEBUG, U1 RP2354A, U2 MCP1702T-3302E_CB, X1 IQXO-791_12MHz

Commit message: Add files via upload
Updated PCB layout
Parts:
- moved C15 29.9 mm to (108.7, 86.2), turned to 90 degrees
- moved C1 29.0 mm to (100.7, 110.1), turned to 90 degrees
- moved D3 28.5 mm to (120.4, 88.6), turned to 180 degrees
- moved U2 28.4 mm to (111.6, 86.2)
- moved C4 26.9 mm to (98.5, 101.1)
- moved C3 25.3 mm to (98.6, 96.2)
- moved C5 24.9 mm to (103.2, 105.8), turned to 90 degrees
- moved R12 24.0 mm to (117.0, 88.6), turned to 0 degrees
- moved S1 22.1 mm to (108.5, 125.6)
- moved C14 19.7 mm to (111.1, 98.5), turned to 180 degrees
- moved R1 18.9 mm to (113.6, 123.4)
- moved C2 18.3 mm to (109.0, 89.3), turned to -90 degrees
- moved C6 16.5 mm to (111.0, 103.6), turned to 180 degrees
- moved C10 14.7 mm to (106.3, 93.3), turned to -90 degrees
- moved C9 14.0 mm to (103.6, 94.1)
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Routing:
- net +5V: track 129.8 -> 28.6 mm, vias 0 -> 4
- net GND: track 103.6 -> 25.1 mm, vias 24 -> 29
- net /RUN: track 78.9 -> 59.9 mm
- net /BOOT: track 40.2 -> 25.7 mm
- net /SWDIO: track 9.44 -> 16.1 mm
- net /GPIO26: track 24.0 -> 18.2 mm
- net /GPIO7: track 16.9 -> 11.6 mm
- net /GPIO4: track 23.1 -> 17.8 mm
- net /GPIO9: track 18.5 -> 13.3 mm
- net /GPIO8: track 17.6 -> 12.4 mm
- net /GPIO25: track 2.67 -> 7.82 mm
- net /GPIO5: track 20.9 -> 15.8 mm
- net /GPIO6: track 17.7 -> 12.6 mm
- net Net-(U1-USB_D+): track 9.37 -> 4.52 mm
- net /GPIO13: track 26.7 -> 21.8 mm
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Other:
- board size 45.7 x 55 mm -> 40.6 x 55 mm
